File: temp_sensor/temp_sensor.kicad_pcb (KiCad board)
At the start: 2 copper layers, 25.5 x 25.5 mm, 9 parts, among them J1 INTERFACE, J2 CC1101, SW1 NRST, U1 STM32G070KBTx, U2 DS18B20

Commit message: Refactor
Parts:
- added R2: 1M, Resistor_SMD:R_1206_3216Metric, F.Cu at (169.1, 93.4)
- R1: footprint Resistor_THT:R_Axial_DIN0207_L6.3mm_D2.5mm_P2.54mm_Vertical -> Resistor_SMD:R_1206_3216Metric
- turned C1 to -90 degrees
Connections:
- J1 pad 7: unconnected-(J1-Pin_7-Pad7) -> VDD
- J2 pad 7: Net-(J2-Pin_7) -> GND
- U1 pad 10: Net-(J2-Pin_7) -> unconnected-(U1-PA3-Pad10)
- U1 pad 11: Net-(J2-Pin_7) -> unconnected-(U1-PA4-Pad11)
- U1 pad 7: VDD -> unconnected-(U1-PA0-Pad7)
Routing:
- net Net-(J2-Pin_7): track 19.6 -> 0.00 mm, vias 1 -> 0
- net VDD: track 28.9 -> 12.3 mm, vias 1 -> 2
- net GND: track 23.2 -> 14.5 mm, vias 1 -> 2
- net Net-(J2-Pin_1): track 20.4 -> 24.1 mm
- net Net-(U1-PA5): track 17.7 -> 19.3 mm, vias 1 -> 2
Other:
- board text added: "GND"
- board text added: "RX"
- board text added: "SWCLK"
- board text added: "SWDIO"
- board text added: "TEMPERATURE SENSOR (c)rsta 2024-03-09"
- board text added: "TX"
- board text added: "VDD"
- board text removed: "temp sensor rsta 2.1.2024"

Commit message: v2
Parts:
- J2: footprint Connector_PinHeader_1.27mm:PinHeader_1x08_P1.27mm_Vertical -> Connector_PinSocket_2.00mm:PinSocket_1x08_P2.00mm_Vertical
- moved J2 3.13 mm to (147.9, 85.4)
- moved C2 1.01 mm to (149.5, 82.1)
Routing:
- net VDD: track 12.3 -> 26.2 mm, vias 2 -> 3
- net GND: track 14.5 -> 23.1 mm, vias 2 -> 3
- net Net-(J2-Pin_1): track 24.1 -> 26.7 mm
- net Net-(J2-Pin_6): track 16.8 -> 17.6 mm
- added copper zone on B.Cu, net VDD
Other:
- board text added: "TEMPERATURE SENSOR (c)rsta 2024-07-22"
- board text removed: "TEMPERATURE SENSOR (c)rsta 2024-03-09"
