File: temp_sensor/temp_sensor.kicad_sch (KiCad schematic)
At the start: 9 parts, among them J1 INTERFACE, J2 CC1101, SW1 NRST, U1 STM32G070KBTx, U2 DS18B20

Commit message: Refactor
Parts:
- added R2: 1M, Resistor_SMD:R_1206_3216Metric, symbol Device:R
- R1: footprint Resistor_THT:R_Axial_DIN0207_L6.3mm_D2.5mm_P2.54mm_Vertical -> Resistor_SMD:R_1206_3216Metric
Connections:
- net GND: now also J2.7 (Pin_7)
- net VDD: now also J1.7 (Pin_7), R2.2; no longer U1.7 (PA0)
- net at J2.1 (Pin_1), U1.14 (PA7): now also R2.1
- now unconnected: U1.10 (PA3), U1.11 (PA4)
Other:
- note added: "GND"
- note added: "RX"
- note added: "SWDCLK"
- note added: "SWDIO"
- note added: "TX"
- note added: "VDD"
Changed lines of the file:
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@@
     (rev "0.9")
   )
+  (junction (at 186.69 41.91) (diameter 0) (color 0 0 0 0)
+  )
   (junction (at 195.58 99.06) (diameter 0) (color 0 0 0 0)
   )
-  (junction (at 167.64 54.61) (diameter 0) (color 0 0 0 0)
-  )
   (junction (at 93.98 54.61) (diameter 0) (color 0 0 0 0)
   )
   (junction (at 154.94 92.71) (diameter 0) (color 0 0 0 0)
   )
+  (junction (at 190.5 67.31) (diameter 0) (color 0 0 0 0)
+  )
   (junction (at 156.21 99.06) (diameter 0) (color 0 0 0 0)
   )
@@
   (junction (at 125.73 113.03) (diameter 0) (color 0 0 0 0)
   )
+  (junction (at 193.04 41.91) (diameter 0) (color 0 0 0 0)
+  )
+  (junction (at 182.88 99.06) (diameter 0) (color 0 0 0 0)
+  )
   (junction (at 104.14 57.15) (diameter 0) (color 0 0 0 0)
   )
   (junction (at 93.98 46.99) (diameter 0) (color 0 0 0 0)
   )
-  (junction (at 177.8 41.91) (diameter 0) (color 0 0 0 0)
-  )
   (junction (at 93.98 85.09) (diameter 0) (color 0 0 0 0)
   )
   (junction (at 93.98 44.45) (diameter 0) (color 0 0 0 0)
   )
-  (wire (pts (xy 179.07 54.61) (xy 179.07 55.88))
-    (stroke (width 0) (type default))
-  )
   (wire (pts (xy 195.58 93.98) (xy 191.77 93.98))
     (stroke (width 0) (type default))
   )
+  (wire (pts (xy 172.72 59.69) (xy 194.31 59.69))
+    (stroke (width 0) (type default))
+  )
   (wire (pts (xy 170.18 59.69) (xy 170.18 104.14))
     (stroke (width 0) (type default))
@@
     (stroke (width 0) (type default))
   )
-  (wire (pts (xy 167.64 54.61) (xy 167.64 57.15))
+  (wire (pts (xy 190.5 77.47) (xy 207.01 77.47))
     (stroke (width 0) (type default))
   )
@@
     (stroke (width 0) (type default))
   )
+  (wire (pts (xy 193.04 41.91) (xy 186.69 41.91))
+    (stroke (width 0) (type default))
+  )
+  (wire (pts (xy 190.5 67.31) (xy 194.31 67.31))
+    (stroke (width 0) (type default))
+  )
   (wire (pts (xy 83.82 54.61) (xy 93.98 54.61))
     (stroke (width 0) (type default))
@@
     (stroke (width 0) (type default))
   )
+  (wire (pts (xy 187.96 69.85) (xy 187.96 88.9))
+    (stroke (width 0) (type default))
+  )
   (wire (pts (xy 177.8 49.53) (xy 167.64 49.53))
     (stroke (width 0) (type default))
@@
     (stroke (width 0) (type default))
   )
-  (wire (pts (xy 167.64 46.99) (xy 177.8 46.99))
-    (stroke (width 0) (type default))
-  )
   (wire (pts (xy 93.98 46.99) (xy 105.41 46.99))
     (stroke (width 0) (type default))
@@
     (stroke (width 0) (type default))
   )
-  (wire (pts (xy 194.31 67.31) (xy 172.72 67.31))
+  (wire (pts (xy 194.31 52.07) (xy 182.88 52.07))
     (stroke (width 0) (type default))
   )
@@
     (stroke (width 0) (type default))
   )
-  (wire (pts (xy 194.31 41.91) (xy 177.8 41.91))
-    (stroke (width 0) (type default))
-  )
-  (wire (pts (xy 177.8 46.99) (xy 177.8 41.91))
+  (wire (pts (xy 194.31 41.91) (xy 193.04 41.91))
+    (stroke (width 0) (type default))
+  )
+  (wire (pts (xy 182.88 99.06) (xy 195.58 99.06))
+    (stroke (width 0) (type default))
+  )
+  (wire (pts (xy 186.69 36.83) (xy 186.69 41.91))
     (stroke (width 0) (type default))
   )
@@
     (stroke (width 0) (type default))
   )
+  (wire (pts (xy 193.04 86.36) (xy 193.04 41.91))
+    (stroke (width 0) (type default))
+  )
   (wire (pts (xy 146.05 104.14) (xy 146.05 113.03))
     (stroke (width 0) (type default))
@@
     (stroke (width 0) (type default))
   )
+  (wire (pts (xy 207.01 36.83) (xy 186.69 36.83))
+    (stroke (width 0) (type default))
+  )
   (wire (pts (xy 156.21 99.06) (xy 154.94 99.06))
     (stroke (width 0) (type default))
@@
     (stroke (width 0) (type default))
   )
-  (wire (pts (xy 194.31 59.69) (xy 172.72 59.69))
-    (stroke (width 0) (type default))
-  )
-  (wire (pts (xy 191.77 55.88) (xy 191.77 52.07))
+  (wire (pts (xy 182.88 52.07) (xy 182.88 99.06))
+    (stroke (width 0) (type default))
+  )
+  (wire (pts (xy 172.72 67.31) (xy 190.5 67.31))
     (stroke (width 0) (type default))
   )
@@
     (stroke (width 0) (type default))
   )
-  (wire (pts (xy 191.77 52.07) (xy 194.31 52.07))
+  (wire (pts (xy 207.01 77.47) (xy 207.01 36.83))
     (stroke (width 0) (type default))
   )
@@
     (stroke (width 0) (type default))
   )
-  (wire (pts (xy 195.58 99.06) (xy 156.21 99.06))
+  (wire (pts (xy 156.21 99.06) (xy 182.88 99.06))
     (stroke (width 0) (type default))
   )
@@
     (stroke (width 0) (type default))
   )
-  (wire (pts (xy 167.64 54.61) (xy 179.07 54.61))
-    (stroke (width 0) (type default))
-  )
   (wire (pts (xy 191.77 80.01) (xy 167.64 80.01))
     (stroke (width 0) (type default))
   )
-  (wire (pts (xy 187.96 69.85) (xy 187.96 88.9))
-    (stroke (width 0) (type default))
-  )
   (wire (pts (xy 185.42 72.39) (xy 185.42 91.44))
     (stroke (width 0) (type default))
   )
+  (wire (pts (xy 195.58 86.36) (xy 193.04 86.36))
+    (stroke (width 0) (type default))
+  )
   (wire (pts (xy 93.98 54.61) (xy 105.41 54.61))
     (stroke (width 0) (type default))
@@
     (stroke (width 0) (type default))
   )
-  (wire (pts (xy 177.8 41.91) (xy 154.94 41.91))
+  (wire (pts (xy 190.5 67.31) (xy 190.5 69.85))
+    (stroke (width 0) (type default))
+  )
+  (wire (pts (xy 154.94 41.91) (xy 186.69 41.91))
     (stroke (width 0) (type default))
   )
@@
     (stroke (width 0) (type default))
   )
-  (wire (pts (xy 179.07 55.88) (xy 191.77 55.88))
-    (stroke (width 0) (type default))
-  )
   (wire (pts (xy 139.7 46.99) (xy 129.54 46.99))
     (stroke (width 0) (type default))
+  )
+  (text "GND" (at 184.15 99.06 0)
+    (effects (font (size 0.8 0.8)) (justify left bottom))
+  )
+  (text "VDD" (at 193.04 86.36 0)
+    (effects (font (size 0.8 0.8)) (justify left bottom))
+  )
+  (text "RX" (at 191.77 91.44 0)
+    (effects (font (size 0.8 0.8)) (justify left bottom))
+  )
+  (text "SWDIO" (at 191.77 93.98 0)
+    (effects (font (size 0.8 0.8)) (justify left bottom))
+  )
+  (text "TX" (at 191.77 88.9 0)
+    (effects (font (size 0.8 0.8)) (justify left bottom))
+  )
+  (text "SWDCLK" (at 191.77 96.52 0)
+    (effects (font (size 0.8 0.8)) (justify left bottom))
   )
   (symbol (lib_id "power:GND") (at 93.98 58.42 0) (unit 1)
@@
       (effects (font (size 1.27 1.27)))
     )
-    (property "Footprint" "Resistor_THT:R_Axial_DIN0207_L6.3mm_D2.5mm_P2.54mm_Vertical" (at 138.43 114.808 90)
+    (property "Footprint" "Resistor_SMD:R_1206_3216Metric" (at 138.43 114.808 90)
       (effects (font (size 1.27 1.27)) hide)
     )
@@
         )
       )
+    )
+  )
+  (symbol (lib_id "Device:R") (at 190.5 73.66 0) (unit 1)
+    (in_bom yes) (on_board yes) (dnp no) (fields_autoplaced)
+    (property "Reference" "R2" (at 193.04 72.39 0)
+      (effects (font (size 1.27 1.27)) (justify left))
+    )
+    (property "Value" "1M" (at 193.04 74.93 0)
+      (effects (font (size 1.27 1.27)) (justify left))
+    )
+    (property "Footprint" "Resistor_SMD:R_1206_3216Metric" (at 188.722 73.66 90)
+      (effects (font (size 1.27 1.27)) hide)
+    )
+    (property "Datasheet" "~" (at 190.5 73.66 0)
+      (effects (font (size 1.27 1.27)) hide)
+    )
+    (pin "1")
+    (pin "2")
+    (instances
+      (project "temp_sensor"
+        (path "/62fc7310-0501-46dd-8802-481846d082e8"
+          (reference "R2") (unit 1)
+        )
+      )

Commit message: v2
Parts:
- J2: footprint Connector_PinHeader_1.27mm:PinHeader_1x08_P1.27mm_Vertical -> Connector_PinSocket_2.00mm:PinSocket_1x08_P2.00mm_Vertical
Changed lines of the file:
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@@
       (effects (font (size 1.27 1.27)))
     )
-    (property "Footprint" "Connector_PinHeader_1.27mm:PinHeader_1x08_P1.27mm_Vertical" (at 199.39 59.69 0)
+    (property "Footprint" "Connector_PinSocket_2.00mm:PinSocket_1x08_P2.00mm_Vertical" (at 199.39 59.69 0)
       (effects (font (size 1.27 1.27)) hide)
     )
