File: sensors_hub/sensors_hub.kicad_pcb (KiCad board)
At the start: 2 copper layers, 65.9 x 30.8 mm, 19 parts, among them J1 INTERFACE, J2 RPi_GPIO, J3 CC1101, J5 Relay, Q1 BS170, SW1 SW_Push, U1 STM32G081KBTx, U2 AMS1117-3.3

Commit message: sensors_hub
Parts:
- J4: footprint TerminalBlock_TE-Connectivity:TerminalBlock_TE_282834-4_1x04_P2.54mm_Horizontal -> TerminalBlock:TerminalBlock_bornier-4_P5.08mm
- moved ? 50.2 mm to (25.3, 63.1)
- moved ? 12.2 mm to (16.7, 63.2)
- moved J4 7.57 mm to (73.0, 51.1)
Connections:
- J4 pad 1: Net-(J4-Pin_1) -> GND
- J4 pad 2: GND -> Net-(J4-Pin_2)
- U1 pad 12: Net-(J4-Pin_1) -> Net-(J4-Pin_2)
Routing:
- net Net-(J4-Pin_2): track 0.00 -> 52.4 mm, vias 0 -> 2
- net Net-(J4-Pin_1): track 50.8 -> 0.00 mm, vias 2 -> 0
- net GND: track 143.0 -> 129.9 mm
- net Net-(J4-Pin_3): track 27.4 -> 30.3 mm
- net Net-(J4-Pin_4): track 12.7 -> 14.0 mm
- added copper zone on F.Cu, net +3.3V
- added copper zone on B.Cu, net GND
Other:
- board text added: "GND"
- board text added: "RX"
- board text added: "SWCLK"
- board text added: "SWDIO"
- board text added: "TX"
- board text added: "VDD"
- board text added: "sensors-hub (c) rsta 240920"
