File: sensors_hub/sensors_hub.kicad_sch (KiCad schematic)
At the start: 15 parts, among them J1 INTERFACE, J2 RPi_GPIO, J3 CC1101, J5 Relay, Q1 BS170, SW1 SW_Push, U1 STM32G081KBTx, U2 AMS1117-3.3

Commit message: sensors_hub
Parts:
- J4: footprint TerminalBlock_TE-Connectivity:TerminalBlock_TE_282834-4_1x04_P2.54mm_Horizontal -> TerminalBlock:TerminalBlock_bornier-4_P5.08mm
- Q1: value BS170 -> 2N7000
Connections:
- net GND: now also J4.1 (Pin_1); no longer J4.2 (Pin_2)
- net at U1.12 (PA5): now also J4.2 (Pin_2); no longer J4.1 (Pin_1)
Changed lines of the file:
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@@
+    (stroke (width 0) (type default))
+  )
+  (wire (pts (xy 162.56 92.71) (xy 162.56 90.17))
     (stroke (width 0) (type default))
   )
@@
     (stroke (width 0) (type default))
   )
-  (wire (pts (xy 165.1 38.1) (xy 165.1 90.17))
+  (wire (pts (xy 165.1 38.1) (xy 165.1 92.71))
     (stroke (width 0) (type default))
   )
@@
     (stroke (width 0) (type default))
   )
+  (wire (pts (xy 165.1 92.71) (xy 177.8 92.71))
+    (stroke (width 0) (type default))
+  )
   (wire (pts (xy 170.18 33.02) (xy 170.18 48.26))
     (stroke (width 0) (type default))
@@
     (stroke (width 0) (type default))
   )
+  (wire (pts (xy 162.56 90.17) (xy 177.8 90.17))
+    (stroke (width 0) (type default))
+  )
   (wire (pts (xy 119.38 74.93) (xy 119.38 63.5))
     (stroke (width 0) (type default))
@@
     (stroke (width 0) (type default))
   )
-  (wire (pts (xy 165.1 90.17) (xy 177.8 90.17))
-    (stroke (width 0) (type default))
-  )
   (wire (pts (xy 53.34 85.09) (xy 54.61 85.09))
     (stroke (width 0) (type default))
@@
     (stroke (width 0) (type default))
   )
+  (wire (pts (xy 160.02 92.71) (xy 162.56 92.71))
+    (stroke (width 0) (type default))
+  )
   (wire (pts (xy 40.64 27.94) (xy 46.99 27.94))
     (stroke (width 0) (type default))
@@
   )
   (wire (pts (xy 175.26 20.32) (xy 175.26 30.48))
-    (stroke (width 0) (type default))
-  )
-  (wire (pts (xy 160.02 92.71) (xy 177.8 92.71))
     (stroke (width 0) (type default))
   )
@@
       (effects (font (size 1.27 1.27)))
     )
-    (property "Value" "BS170" (at 147.32 123.19 90)
+    (property "Value" "2N7000" (at 147.32 123.19 90)
       (effects (font (size 1.27 1.27)))
     )
@@
       (effects (font (size 1.27 1.27)) (justify left))
     )
-    (property "Footprint" "TerminalBlock_TE-Connectivity:TerminalBlock_TE_282834-4_1x04_P2.54mm_Horizontal" (at 182.88 92.71 0)
-      (effects (font (size 1.27 1.27)) hide)
-    )
+    (property "Footprint" "TerminalBlock:TerminalBlock_bornier-4_P5.08mm" (at 182.88 92.71 0)
+      (effects (font (size 1.27 1.27)) hide)
+    )
