File: kamil/kamil.kicad_sch (KiCad schematic)
At the start: 33 parts, among them J1 RELAY, J2 RELAY OUTPUT, J3 CC1101, J4 DEBUG INTERFACE, J5 230AC, J6 LED, Q2 2N7000, SW1 SW_Push, U1 LNK304P, U2 AMS1117-3.3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

Commit message: Kamil...
Parts:
- L1, L2: footprint (none) -> Inductor_THT:L_Radial_D10.5mm_P5.00mm_Abacron_AISR-01
- R7: value 10R -> 100K
Changed lines of the file:
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@@
       (effects (font (size 1.27 1.27)))
     )
-    (property "Footprint" "" (at 59.69 58.42 0)
+    (property "Footprint" "Inductor_THT:L_Radial_D10.5mm_P5.00mm_Abacron_AISR-01" (at 59.69 58.42 0)
       (effects (font (size 1.27 1.27)) hide)
     )
@@
       (effects (font (size 1.27 1.27)))
     )
-    (property "Value" "10R" (at 107.95 163.83 90)
+    (property "Value" "100K" (at 107.95 163.83 90)
       (effects (font (size 1.27 1.27)))
     )
@@
       (effects (font (size 1.27 1.27)))
     )
-    (property "Footprint" "" (at 138.43 58.42 0)
-      (effects (font (size 1.27 1.27)) hide)
-    )
+    (property "Footprint" "Inductor_THT:L_Radial_D10.5mm_P5.00mm_Abacron_AISR-01" (at 138.43 58.42 0)
+      (effects (font (size 1.27 1.27)) hide)
+    )

Commit message: Implementation
Connections:
- net +5V: now also J1.2 (Pin_2); no longer J1.3 (Pin_3)
- net at J1.11 (Pin_11): no longer Q2.3 (S)
- net at J1.13 (Pin_13): no longer J2.1 (Pin_1)
- net at J1.6 (Pin_6): now also Q2.3 (S)
- net at J1.7 (Pin_7): now also J2.1 (Pin_1)
Changed lines of the file:
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@@
+    (stroke (width 0) (type default))
+  )
+  (wire (pts (xy 113.03 193.04) (xy 113.03 168.91))
     (stroke (width 0) (type default))
   )
@@
     (stroke (width 0) (type default))
   )
-  (wire (pts (xy 128.27 181.61) (xy 128.27 194.31))
-    (stroke (width 0) (type default))
-  )
   (wire (pts (xy 111.76 58.42) (xy 124.46 58.42))
     (stroke (width 0) (type default))
@@
     (stroke (width 0) (type default))
   )
-  (wire (pts (xy 96.52 194.31) (xy 128.27 194.31))
-    (stroke (width 0) (type default))
-  )
   (wire (pts (xy 163.83 58.42) (xy 172.72 58.42))
     (stroke (width 0) (type default))
@@
     (stroke (width 0) (type default))
   )
-  (wire (pts (xy 118.11 181.61) (xy 118.11 196.85))
-    (stroke (width 0) (type default))
-  )
   (wire (pts (xy 111.76 119.38) (xy 111.76 113.03))
     (stroke (width 0) (type default))
@@
     (stroke (width 0) (type default))
   )
+  (wire (pts (xy 113.03 168.91) (xy 115.57 168.91))
+    (stroke (width 0) (type default))
+  )
   (wire (pts (xy 163.83 68.58) (xy 184.15 68.58))
     (stroke (width 0) (type default))
@@
     (stroke (width 0) (type default))
   )
+  (wire (pts (xy 123.19 189.23) (xy 139.7 189.23))
+    (stroke (width 0) (type default))
+  )
   (wire (pts (xy 85.09 172.72) (xy 85.09 196.85))
     (stroke (width 0) (type default))
@@
     (stroke (width 0) (type default))
   )
+  (wire (pts (xy 134.62 194.31) (xy 134.62 166.37))
+    (stroke (width 0) (type default))
+  )
   (wire (pts (xy 123.19 39.37) (xy 124.46 39.37))
     (stroke (width 0) (type default))
@@
     (stroke (width 0) (type default))
   )
-  (wire (pts (xy 130.81 189.23) (xy 139.7 189.23))
-    (stroke (width 0) (type default))
-  )
   (wire (pts (xy 184.15 58.42) (xy 184.15 59.69))
     (stroke (width 0) (type default))
@@
     (stroke (width 0) (type default))
   )
+  (wire (pts (xy 134.62 166.37) (xy 120.65 166.37))
+    (stroke (width 0) (type default))
+  )
   (wire (pts (xy 19.05 123.19) (xy 26.67 123.19))
     (stroke (width 0) (type default))
@@
     (stroke (width 0) (type default))
   )
+  (wire (pts (xy 96.52 194.31) (xy 134.62 194.31))
+    (stroke (width 0) (type default))
+  )
   (wire (pts (xy 180.34 58.42) (xy 184.15 58.42))
     (stroke (width 0) (type default))
@@
     (stroke (width 0) (type default))
   )
-  (wire (pts (xy 130.81 181.61) (xy 130.81 189.23))
-    (stroke (width 0) (type default))
-  )
   (wire (pts (xy 132.08 128.27) (xy 132.08 101.6))
     (stroke (width 0) (type default))
@@
     (stroke (width 0) (type default))
   )
+  (wire (pts (xy 118.11 196.85) (xy 118.11 193.04))
+    (stroke (width 0) (type default))
+  )
   (wire (pts (xy 148.59 149.86) (xy 148.59 151.13))
     (stroke (width 0) (type default))
@@
     (stroke (width 0) (type default))
   )
+  (wire (pts (xy 120.65 166.37) (xy 120.65 168.91))
+    (stroke (width 0) (type default))
+  )
   (wire (pts (xy 153.67 52.07) (xy 153.67 58.42))
     (stroke (width 0) (type default))
@@
     (stroke (width 0) (type default))
   )
+  (wire (pts (xy 123.19 189.23) (xy 123.19 181.61))
+    (stroke (width 0) (type default))
+  )
   (wire (pts (xy 29.21 77.47) (xy 29.21 58.42))
     (stroke (width 0) (type default))
@@
     (stroke (width 0) (type default))
   )
+  (wire (pts (xy 118.11 193.04) (xy 113.03 193.04))
+    (stroke (width 0) (type default))
+  )
